File: KiCAD/eggtimer.kicad_pcb (KiCad board)
At the start: 2 copper layers, 39 parts, among them SW2 RotaryEncoder, SW3 SW_Push_DPDT, U1 STM32F042F6Px, U2 MCP73831-2-MC, U3 MCP1700x-330xxMB

Commit message: Add files via upload
Parts:
- added BZ1: Buzzer, custom:HND-2319 Buzzer, F.Cu at (95.5, 82.0)
- added J1: USB_C_Receptacle_USB2.0_16P, Connector_USB:USB_C_Receptacle_GCT_USB4105-xx-A_16P_TopMnt_Horizontal, F.Cu at (69.9, 55.0)
- added J3: Conn_01x05_Pin, Connector_Harwin:Harwin_LTek-Male_05_P2.00mm_Vertical, F.Cu at (106.0, 39.0)
- added U4: 74HC595, custom:74HC595D,118 SOIC-16 Shift Registers, F.Cu at (106.5, 66.7)
- D1: renamed from D9; value LED white/yellow -> LED white
- D2: renamed from D12; value LED white/yellow -> LED white
- D3: renamed from D10; value LED white/yellow -> LED white
- D4: renamed from D13; value LED white/yellow -> LED white
- D5: renamed from D11; value LED white/yellow -> LED white
- D6: renamed from D3; value LED white/yellow -> LED white
- D7: renamed from D2; value LED white/yellow -> LED white
- D8: renamed from D4; value LED white/yellow -> LED white
- moved SW2 106.6 mm to (75.8, 71.2)
- moved C10 95.5 mm to (84.5, 54.0), turned to 90 degrees
- moved C3 86.7 mm to (88.0, 59.5)
- moved U2 82.3 mm to (85.6, 50.7)
- moved U3 79.4 mm to (106.8, 54.2)
- moved SW3 77.9 mm to (98.8, 52.4), turned to 90 degrees
- moved R4 74.8 mm to (93.0, 51.4), turned to 90 degrees
- moved R10 64.9 mm to (90.0, 47.9), turned to -90 degrees
- moved R3 62.8 mm to (88.3, 47.9), turned to -90 degrees
- moved D9 61.6 mm to (90.5, 51.4), turned to 180 degrees
- moved R8 61.1 mm to (86.4, 62.4), turned to -90 degrees
- moved R9 60.0 mm to (88.1, 65.9), turned to 90 degrees
- moved R1 59.5 mm to (76.2, 51.2), turned to 180 degrees
- moved C8 56.8 mm to (83.8, 64.2), turned to 90 degrees
- moved C9 56.6 mm to (84.3, 66.2)
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- renumbered D1 to D9
Routing:
- net +3.3V: track 0.00 -> 73.8 mm, vias 0 -> 4
- net GND: track 0.00 -> 56.0 mm, vias 0 -> 13
- net Net-(J3-Pin_2): track 0.00 -> 30.9 mm, vias 0 -> 1
- net Net-(U1-PA0): track 0.00 -> 28.5 mm
- net D+: track 0.00 -> 28.4 mm
- net D-: track 0.00 -> 28.1 mm, vias 0 -> 2
- net nrst: track 0.00 -> 27.1 mm, vias 0 -> 1
- net Net-(J3-Pin_4): track 0.00 -> 25.8 mm, vias 0 -> 1
- net Net-(U1-PA1): track 0.00 -> 22.4 mm
- net Net-(D1-A): track 0.00 -> 21.2 mm
- net +5V: track 0.00 -> 20.6 mm
- net +BATT: track 0.00 -> 18.9 mm
- net Net-(BZ1-+): track 0.00 -> 11.8 mm
- net reg: track 0.00 -> 9.29 mm
- net Net-(D8-A): track 0.00 -> 8.78 mm
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- added copper zone on B.Cu, net GND

Commit message: Add files via upload
KiCAD: need to fix BOM
Parts:
- added Battery_Cell1: Battery_Cell, custom:screw_terminal_2, F.Cu at (115.0, 52.0)
- added D10: LED G, LED_SMD:LED_0805_2012Metric, F.Cu at (100.2, 45.0)
- added H1: M_H, MountingHole:MountingHole_2.2mm_M2, F.Cu at (119.0, 89.0)
- added H2: M_H, MountingHole:MountingHole_2.2mm_M2, F.Cu at (70.0, 89.0)
- added H3: M_H, MountingHole:MountingHole_2.2mm_M2, F.Cu at (70.0, 45.0)
- added H4: M_H, MountingHole:MountingHole_2.2mm_M2, F.Cu at (119.0, 45.0)
- added R11: 680, Resistor_SMD:R_0402_1005Metric, F.Cu at (103.7, 44.3)
- added R17: 680, Resistor_SMD:R_0402_1005Metric, F.Cu at (93.9, 51.4)
- added R18: 680, Resistor_SMD:R_0402_1005Metric, F.Cu at (103.7, 45.7)
- added egg: LOGO, LOGO, F.Cu at (113.0, 84.0)
- D1, D2, D3, D4, D5, D6, D7, D8: value LED white -> LED yellow
- D9: value LED GREEN -> LED r
- MCP1700: renamed from U3; value MCP1700x-330xxMB -> ~
- Push_Button1: renamed from SW3; value SW_Push_DPDT -> SW_Push
- R12, R13, R14, R15, R16, R4, R5, R6, R7: value 330 -> 680
- Rotary_Encoder1: renamed from SW2; value RotaryEncoder -> Rotary_Encoder
- nrst-swclk-gnd-swdio-3v3: renamed from J3; value Conn_01x05_Pin -> nrst swclk gnd swdio 3v3
- moved nrst-swclk-gnd-swdio-3v3 22.7 mm to (84.5, 46.3)
- moved D9 4.38 mm to (94.3, 49.2), turned to 90 degrees
- moved C6 4.03 mm to (89.2, 47.5), turned to 90 degrees
- moved Buzzer1 3.21 mm to (95.8, 78.8)
- moved R10 2.65 mm to (92.5, 48.9)
- moved R3 2.65 mm to (90.8, 48.9)
- moved Rotary_Encoder1 2.60 mm to (75.7, 68.6)
- moved D6 2.57 mm to (114.1, 62.9)
- moved D7 2.57 mm to (114.1, 60.4)
- moved D8 2.57 mm to (114.1, 57.9)
- moved D1 2.57 mm to (114.1, 75.4)
- moved D2 2.57 mm to (114.1, 72.9)
- moved D3 2.57 mm to (114.1, 70.4)
- moved D4 2.57 mm to (114.1, 67.9)
- moved D5 2.57 mm to (114.1, 65.4)
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- renumbered U4 to 74HC595, BZ1 to Buzzer1, U1 to STM32F042F6P6
Connections:
- net Net-(J3-Pin_2) renamed /SWDIO
- net Net-(J3-Pin_4) renamed /SWCLK
- D9 pad 2: Net-(D9-A) -> +5V
- R4 pad 1: GND -> Net-(R17-Pad2)
- R4 pad 2: Net-(D9-K) -> Net-(U2-STAT)
- U2 pad 5: Net-(D9-A) -> Net-(U2-STAT)
Routing:
- net +BATT: track 18.9 -> 32.5 mm, vias 0 -> 1
- net /SWDIO: track 30.9 -> 21.2 mm
- net +5V: track 20.6 -> 27.0 mm
- net Net-(74HC595-QE): track 7.25 -> 3.08 mm
- net Net-(74HC595-QF): track 7.76 -> 3.59 mm
- net Net-(74HC595-QG): track 8.27 -> 4.44 mm
- net Net-(74HC595-QD): track 6.74 -> 3.28 mm
- net Net-(D10-K): track 0.00 -> 3.31 mm
- net Net-(74HC595-QH): track 8.78 -> 5.67 mm
- net Net-(74HC595-QC): track 6.65 -> 3.79 mm
- net reg: track 9.29 -> 12.0 mm
- net Net-(D9-A): track 2.69 -> 0.00 mm
- net Net-(74HC595-QB): track 7.16 -> 4.53 mm
- net Net-(Buzzer1-+): track 11.8 -> 9.32 mm
- net Net-(STM32F042F6P6-PA1): track 22.4 -> 20.2 mm
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Other:
- board outline added: 55 x 50 mm
- board text added: "Eggtimer 2026-06-17"

Commit message: final
Parts:
- removed MCP1700: ~, Package_TO_SOT_SMD:SOT-89-3
- added HT7533-1: ~, Package_TO_SOT_SMD:SOT-89-3, F.Cu at (107.4, 53.4)
- added U1: USBLC6-2SC6, Package_TO_SOT_SMD:SOT-23-6, F.Cu at (80.7, 54.9)
- nrst-swclk-gnd-swdio-3v3: value nrst swclk gnd swdio 3v3 -> nrst-swclk-gnd-swdio-3v3
- moved Buzzer1 0.55 mm to (95.8, 79.3)
- moved C4 0.33 mm to (98.8, 63.0)
- renumbered Push_Button1 to Button
Connections:
- J1 pad A6: D+ -> /usb_d+
- J1 pad A7: D- -> /usb_d-
- J1 pad B6: D+ -> /usb_d+
- J1 pad B7: D- -> /usb_d-
Routing:
- net /usb_d-: track 0.00 -> 12.1 mm
- net +5V: track 27.0 -> 38.4 mm
- net /usb_d+: track 0.00 -> 11.2 mm, vias 0 -> 2
- net GND: track 53.8 -> 62.9 mm, vias 11 -> 16
- net +BATT: track 32.5 -> 39.6 mm
- net D+: track 28.4 -> 24.2 mm
- net D-: track 28.1 -> 25.4 mm, vias 2 -> 0
- net reg: track 12.0 -> 13.8 mm
- net /SWDIO: track 21.2 -> 22.0 mm
- net /SWCLK: track 24.3 -> 25.1 mm
- net Net-(J1-CC1): track 8.23 -> 7.55 mm
- net +3.3V: track 74.8 -> 75.4 mm
- net Net-(Buzzer1-+): track 9.32 -> 9.87 mm
