File: KiCAD/eggtimer.kicad_sch (KiCad schematic)
At the start: 17 parts, among them J1 USB_C_Receptacle_USB2.0_16P, U1 STM32F042F6Px, U2 MCP73831-2-MC, U3 MCP1700x-330xxMB, U4 MCP73871

Commit message: Add files via upload
Parts:
- removed U4: MCP73871, Package_DFN_QFN:QFN-20-1EP_4x4mm_P0.5mm_EP2.5x2.5mm, symbol Battery_Management:MCP73871
- added BZ1: Buzzer, symbol Device:Buzzer
- added C10: 4u7, symbol Device:C
- added SW1: SW_Nidec_CAS-120A1, Button_Switch_SMD:Nidec_Copal_CAS-120A, symbol Switch:SW_Nidec_CAS-120A1
- added SW2: RotaryEncoder, symbol Device:RotaryEncoder
- R3: value R -> 2k
Connections:
- net +BATT: now also C10.2, SW1.1 (C); no longer C1.1, U3.2 (VI)
- net GND: now also C10.1, SW2.C
- net at U1.10 (PA4): now also BZ1.1 (+)
- net at U1.12 (PA6): now also BZ1.2 (-)
- net at U1.6 (PA0): now also SW2.A
- net at U1.8 (PA2): now also SW2.B
- new net reg: C1.1, SW1.2 (B), U3.2 (VI)
- no-connect marks 2 -> 3
Other:
- note added: "check if this is correct also add something to indicate minutes"
- note added: "on off switch from battery to regulator +batt-- I---MCU 5V --"
- note removed: "kanske andvända denna istället"

Commit message: Add files via upload
Parts:
- added C7: 1u, symbol Device:C
- added D10, D11, D12, D13, D2, D3, D4, D9: LED white/yellow, symbol Device:LED
- added J3: Conn_01x05_Pin, symbol Connector:Conn_01x05_Pin
- added R12, R13, R14, R15, R16, R5, R6, R7: 330, symbol Device:R
- added U4: 74HC595, symbol 74xx:74HC595
- C3: value 1u -> 4u7
Connections:
- net +3.3V: now also C7.2, J3.1 (Pin_1), U4.10 (~{SRCLR}), U4.16 (VCC)
- net GND: now also BZ1.2 (-), C7.1, J3.3 (Pin_3), R12.1, R13.1, R14.1, R15.1, R16.1, R5.1, R6.1, R7.1, U4.13 (~{OE}), U4.8 (GND)
- net at U1.10 (PA4): no longer BZ1.1 (+)
- net at U1.11 (PA5): now also U4.14 (SER)
- net at U1.12 (PA6): now also U4.11 (SRCLK); no longer BZ1.2 (-)
- net at U1.13 (PA7): now also U4.12 (RCLK)
- net at U1.19 (PA13): now also J3.2 (Pin_2)
- net at U1.20 (PA14): now also J3.4 (Pin_4)
- net nrst: now reaches U1.4 (NRST)
- net nrst: now also J3.5 (Pin_5)
- net at U1.7 (PA1): now also SW2.B
- net at U1.8 (PA2): now also BZ1.1 (+); no longer SW2.B
- new net: D10.1 (K), R14.2
- new net: D10.2 (A), U4.2 (QC)
- new net: D4.1 (K), R7.2
- new net: D4.2 (A), U4.7 (QH)
- new net: D12.2 (A), U4.1 (QB)
- new net: D9.2 (A), U4.15 (QA)
- new net: D13.2 (A), U4.3 (QD)
- new net: D11.2 (A), U4.4 (QE)
- new net: D3.2 (A), U4.5 (QF)
- new net: D2.2 (A), U4.6 (QG)
- new net: D3.1 (K), R6.2
- new net: D9.1 (K), R12.2
- new net: D12.1 (K), R13.2
- new net: D2.1 (K), R5.2
- new net: D13.1 (K), R15.2
- new net: D11.1 (K), R16.2
- no-connect marks 3 -> 10
Other:
- note added: "HND-2319"
- note added: "Need to fix pcb footprints for encoder, buzzer switch"
- note added: "check if this is correct PEC12R-4220F-N0024 Need pull up resistor and capacitor for filtering"
- note removed: "check if this is correct also add something to indicate minutes"
- moved on the sheet: BZ1, C3, C4, C5, SW2, U1

Commit message: updated schematic
Parts:
- removed SW1: SW_Nidec_CAS-120A1, Button_Switch_SMD:Nidec_Copal_CAS-120A, symbol Switch:SW_Nidec_CAS-120A1
- added C8, C9: 100n, Capacitor_SMD:C_0402_1005Metric, symbol Device:C
- added R10: 5k1, Resistor_SMD:R_0603_1608Metric, symbol Device:R
- added R8, R9: 10k, Resistor_SMD:R_0805_2012Metric, symbol Device:R
- added SW3: SW_Push_DPDT, custom:TK-6580DS-1 push button, symbol Switch:SW_Push_DPDT
- C1, C2, C6, C7: footprint (none) -> Capacitor_SMD:C_0603_1608Metric
- C10, C3: footprint (none) -> Capacitor_SMD:C_0805_2012Metric
- C4, C5: value 1u -> 100n; footprint (none) -> Capacitor_SMD:C_0402_1005Metric
- D1, D10, D11, D12, D13, D2, D3, D4, D9: footprint (none) -> LED_SMD:LED_0805_2012Metric
- R1, R2: footprint (none) -> Resistor_SMD:R_0603_1608Metric
- R12, R13, R14, R15, R16, R4, R5, R6, R7: footprint (none) -> Resistor_SMD:R_0402_1005Metric
- R3: value 2k -> 5k1; footprint (none) -> Resistor_SMD:R_0603_1608Metric
- SW2: footprint (none) -> custom:PEC12R-4220F-N0024 encoder
Connections:
- net +3.3V: now also R8.1, R9.1
- net +BATT: now also SW3.1 (A)
- net GND: now also R3.1, C8.1, C9.1, R10.1; no longer R3.2
- net reg: now also SW3.2 (B)
- net at SW2.A, U1.6 (PA0): now also C8.2, R8.2
- net at SW2.B, U1.7 (PA1): now also C9.2, R9.2
- net at U2.8 (PROG): now also R3.2, R10.2; no longer R3.1
- no-connect marks 10 -> 13
Other:
- note added: "5k1//5k1 aprox 2k5"
- note added: "LED KT-0805G"
- note added: "battery needs footprint"
- note added: "buzzer needs footprint"
- note added: "check if this is correct PEC12R-4220F-N0024"
- note added: "current = 1000mA/prog"
- note added: "encoder needs footprint"
- note added: "on off switch from battery to regulator TK-6580DS-1 need footprint +batt-- I---MCU 5V --"
- note removed: "Need to fix pcb footprints for encoder, buzzer switch"
- note removed: "check if this is correct PEC12R-4220F-N0024 Need pull up resistor and capacitor for filtering"
- note removed: "on off switch from battery to regulator +batt-- I---MCU 5V --"
- moved on the sheet: BZ1

Commit message: pcb: all done except battery, and debug pins
Parts:
- BZ1: footprint (none) -> custom:HND-2319 Buzzer
- D1: renamed from D9; value LED white/yellow -> LED white
- D2: renamed from D12; value LED white/yellow -> LED white
- D3: renamed from D10; value LED white/yellow -> LED white
- D4: renamed from D13; value LED white/yellow -> LED white
- D5: renamed from D11; value LED white/yellow -> LED white
- D6: renamed from D3; value LED white/yellow -> LED white
- D7: renamed from D2; value LED white/yellow -> LED white
- D8: renamed from D4; value LED white/yellow -> LED white
- J1: footprint (none) -> Connector_USB:USB_C_Receptacle_GCT_USB4105-xx-A_16P_TopMnt_Horizontal
- J3: footprint (none) -> Connector_Harwin:Harwin_LTek-Male_05_P2.00mm_Vertical
- U4: footprint (none) -> custom:74HC595D,118 SOIC-16 Shift Registers
- renumbered D1 to D9
Other:
- note removed: "buzzer needs footprint"
- note removed: "encoder needs footprint"
Changed lines of the file:
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@@
 		)
 	)
-	(text "encoder needs footprint"
-		(exclude_from_sim no)
-		(at 269.748 114.3 0)
-		(effects
-			(font
-				(size 1.27 1.27)
-				(thickness 0.254)
-				(bold yes)
-			)
-			(justify left bottom)
-		)
-	)
 	(text "5k1//5k1\naprox 2k5"
 		(exclude_from_sim no)
@@
 		)
 	)
-	(text "buzzer needs footprint"
-		(exclude_from_sim no)
-		(at 276.606 142.748 0)
-		(effects
-			(font
-				(size 1.27 1.27)
-				(thickness 0.254)
-				(bold yes)
-			)
-			(justify left bottom)
-		)
-	)
 	(text "check if this is correct\nPEC12R-4220F-N0024\n\n"
 		(exclude_from_sim no)
@@
 		(on_board yes)
 		(dnp no)
-		(property "Reference" "D10"
+		(property "Reference" "D3"
 			(at 270.51 164.338 0)
 			(effects
@@
 			)
 		)
-		(property "Value" "LED white/yellow"
+		(property "Value" "LED white"
 			(at 273.304 167.132 0)
 			(effects
@@
 			(project "eggtimer"
 				(path "/4b87e02e-73da-44fc-9ee3-219697950739"
-					(reference "D10")
+					(reference "D3")
 					(unit 1)
 				)
@@
 		(on_board yes)
 		(dnp no)
-		(property "Reference" "D4"
+		(property "Reference" "D8"
 			(at 279.4 177.038 0)
 			(effects
@@
 			)
 		)
-		(property "Value" "LED white/yellow"
+		(property "Value" "LED white"
 			(at 282.194 179.832 0)
 			(effects
@@
 			(project "eggtimer"
 				(path "/4b87e02e-73da-44fc-9ee3-219697950739"
-					(reference "D4")
+					(reference "D8")
 					(unit 1)
 				)
@@
 			)
 		)
-		(property "Footprint" ""
+		(property "Footprint" "custom:74HC595D,118  SOIC-16 Shift Registers"
 			(at 255.27 170.18 0)
 			(effects
@@
 		(on_board yes)
 		(dnp no)
-		(property "Reference" "D1"
+		(property "Reference" "D9"
 			(at 238.76 63.5 0)
 			(effects
@@
 			(project "eggtimer"
 				(path "/4b87e02e-73da-44fc-9ee3-219697950739"
-					(reference "D1")
+					(reference "D9")
 					(unit 1)
 				)
@@
 			)
 		)
-		(property "Footprint" ""
+		(property "Footprint" "Connector_Harwin:Harwin_LTek-Male_05_P2.00mm_Vertical"
 			(at 220.98 184.15 0)
 			(effects
@@
 		(on_board yes)
 		(dnp no)
-		(property "Reference" "D12"
+		(property "Reference" "D2"
 			(at 279.4 161.798 0)
 			(effects
@@
 			)
 		)
-		(property "Value" "LED white/yellow"
+		(property "Value" "LED white"
 			(at 282.194 164.592 0)
 			(effects
@@
 			(project "eggtimer"
 				(path "/4b87e02e-73da-44fc-9ee3-219697950739"
-					(reference "D12")
+					(reference "D2")
 					(unit 1)
 				)
@@
 		(on_board yes)
 		(dnp no)
-		(property "Reference" "D9"
+		(property "Reference" "D1"
 			(at 270.51 159.258 0)
 			(effects
@@
 			)
 		)
-		(property "Value" "LED white/yellow"
+		(property "Value" "LED white"
 			(at 273.304 162.052 0)
 			(effects
@@
 			(project "eggtimer"
 				(path "/4b87e02e-73da-44fc-9ee3-219697950739"
-					(reference "D9")
+					(reference "D1")
 					(unit 1)
 				)
@@
 			)
 		)
-		(property "Footprint" ""
+		(property "Footprint" "Connector_USB:USB_C_Receptacle_GCT_USB4105-xx-A_16P_TopMnt_Horizontal"
 			(at 46.99 57.15 0)
 			(effects
@@
 			)
 		)
-		(property "Footprint" ""
+		(property "Footprint" "custom:HND-2319 Buzzer"
 			(at 286.385 130.81 90)
 			(effects
@@
 		(on_board yes)
 		(dnp no)
-		(property "Reference" "D2"
+		(property "Reference" "D7"
 			(at 270.51 174.498 0)
 			(effects
@@
 			)
 		)
-		(property "Value" "LED white/yellow"
+		(property "Value" "LED white"
 			(at 273.304 177.292 0)
 			(effects
@@
 			(project "eggtimer"
 				(path "/4b87e02e-73da-44fc-9ee3-219697950739"
-					(reference "D2")
+					(reference "D7")
 					(unit 1)
 				)
@@
 		(on_board yes)
 		(dnp no)
-		(property "Reference" "D13"
+		(property "Reference" "D4"
 			(at 279.4 166.878 0)
 			(effects
@@
 			)
 		)
-		(property "Value" "LED white/yellow"
+		(property "Value" "LED white"
 			(at 282.194 169.672 0)
 			(effects
@@
 			(project "eggtimer"
 				(path "/4b87e02e-73da-44fc-9ee3-219697950739"
-					(reference "D13")
+					(reference "D4")
 					(unit 1)
 				)
@@
 		(on_board yes)
 		(dnp no)
-		(property "Reference" "D11"
+		(property "Reference" "D5"
 			(at 270.51 169.418 0)
 			(effects
@@
 			)
 		)
-		(property "Value" "LED white/yellow"
+		(property "Value" "LED white"
 			(at 273.304 172.212 0)
 			(effects
@@
 			(project "eggtimer"
 				(path "/4b87e02e-73da-44fc-9ee3-219697950739"
-					(reference "D11")
+					(reference "D5")
 					(unit 1)
 				)
@@
 		(on_board yes)
 		(dnp no)
-		(property "Reference" "D3"
+		(property "Reference" "D6"
 			(at 279.4 171.958 0)
 			(effects
@@
 			)
 		)
-		(property "Value" "LED white/yellow"
+		(property "Value" "LED white"
 			(at 282.194 174.752 0)
 			(effects
@@
 			(project "eggtimer"
 				(path "/4b87e02e-73da-44fc-9ee3-219697950739"
-					(reference "D3")
+					(reference "D6")
 					(unit 1)
 				)

Commit message: Add files via upload
KiCAD: need to fix BOM
Parts:
- added D10: LED G, LED_SMD:LED_0805_2012Metric, symbol Device:LED
- added H1, H2, H3, H4: M_H, MountingHole:MountingHole_2.2mm_M2, symbol Mechanical:MountingHole
- added R11, R17, R18: 680, Resistor_SMD:R_0402_1005Metric, symbol Device:R
- Battery_Cell1: renamed from BT1; footprint (none) -> custom:screw_terminal_2
- D1, D2, D3, D4, D5, D6, D7, D8: value LED white -> LED yellow
- D9: value LED GREEN -> LED r
- MCP1700: renamed from U3; value MCP1700x-330xxMB -> ~
- Push_Button1: renamed from SW3; value SW_Push_DPDT -> SW_Push
- R12, R13, R14, R15, R16, R4, R5, R6, R7: value 330 -> 680
- Rotary_Encoder1: renamed from SW2; value RotaryEncoder -> Rotary_Encoder
- nrst-swclk-gnd-swdio-3v3: renamed from J3; value Conn_01x05_Pin -> nrst swclk gnd swdio 3v3
- renumbered U4 to 74HC595, BZ1 to Buzzer1, U1 to STM32F042F6P6
Connections:
- net +5V: now also D9.2 (A)
- net GND: now also R11.1, R18.1; no longer R4.1
- net reg: now also D10.2 (A)
- net at D9.1 (K): now also R17.1; no longer R4.2
- net at U2.5 (STAT): now also R4.2; no longer D9.2 (A)
- net SWDIO: now reaches STM32F042F6P6.19 (PA13), nrst-swclk-gnd-swdio-3v3.2 (Pin_2)
- net SWCLK: now reaches STM32F042F6P6.20 (PA14), nrst-swclk-gnd-swdio-3v3.4 (Pin_4)
- new net: D10.1 (K), R11.2, R18.2
- new net: R17.2, R4.1
Other:
- note added: "LED KT-0805G 2.6V~3.1V"
- note added: "LED KT-0805R"
- note added: "LEDS KT-0805Y 1.8V~2.4V"
- note added: "battery C5154896 500mAh 3.7V LiPo with protection circuit JST-PH connector optional"
- note removed: "LED KT-0805G"
- note removed: "battery 500mAh 3.7V LiPo with protection circuit JST-PH connector optional"
- note removed: "battery needs footprint"
- moved on the sheet: D9

Commit message: final
Parts:
- removed MCP1700: ~, Package_TO_SOT_SMD:SOT-89-3, symbol Regulator_Linear:MCP1700x-330xxMB
- added MCP1700: ~, Package_TO_SOT_SMD:SOT-89-3, symbol Regulator_Linear:HT75xx-1-SOT89
- added U1: USBLC6-2SC6, Package_TO_SOT_SMD:SOT-23-6, symbol Power_Protection:USBLC6-2SC6
Connections:
- net +3.3V: now also MCP1700.3 (VOUT)
- net +5V: now also U1.5 (VBUS)
- net D+: now also U1.4 (I/O2); no longer J1.A6 (D+), J1.B6 (D+)
- net D-: now also U1.6 (I/O1); no longer J1.A7 (D-), J1.B7 (D-)
- net GND: now also MCP1700.1 (GND), U1.2 (GND)
- net reg: now also MCP1700.2 (VIN)
- new net usb_d+: J1.A6 (D+), J1.B6 (D+), U1.3 (I/O2)
- new net usb_d-: J1.A7 (D-), J1.B7 (D-), U1.1 (I/O1)
Other:
- note added: "NEED TO FIX THIS not mpc take voltage regulator 3.3 v from jlcpcb check all"
